Commit message: [Update]: Added 3 robots to the basement world, lego block moving with box

File: catkin_ws/src/navigation_oru-release/gazebo_oru/cititruck/cititruck_description/urdf/cititruck.xacro (robot description, xacro)
@@ -63,5 +63,5 @@
           <box size="0.8 0.1 0.01" />
         </geometry>
-        <material name="grey" />
+        <material name="brown" />
       </visual>
       <collision>
@@ -85,5 +85,5 @@
           <box size="0.8 0.1 0.01" />
         </geometry>
-        <material name="grey" />
+        <material name="brown" />
       </visual>
       <collision>
@@ -107,5 +107,5 @@
           <box size="0.01 0.01 0.01" />
         </geometry>
-        <material name="grey" />
+        <material name="brown" />
       </visual>
     </link>
