Commit message: checking in the pr2 navigation 1

File: catkin_ws/src/navigation_oru-release/levelManager/models/test.urdf (robot description, URDF)
Before this commit: robot dustbin, 15 links, 14 joints
Links:
- link base_link: geometry collision box size=0.5 0.5 0.15; visual box size=0.5 0.5 0.15
Joints:
- joint handle_joint_l: origin xyz=0.1 0.25 0.2 rpy=0 1.57 0 -> xyz=0.1 0.25 0.07 rpy=0 1.57 0
- joint handle_joint_r: origin xyz=0.1 -0.25 0.2 rpy=0 1.57 0 -> xyz=0.1 -0.25 0.07 rpy=0 1.57 0
